File: EE514 Board/Amplifier.sch (KiCad schematic (older format))
At the start: 12 parts

Commit message: Layout finished, updating silkscreen...
Parts:
- removed J? (x2): SMA, symbol Connector:Conn_Coaxial
- C201, C202, C203, C204, C205: renamed from C?; footprint (none) -> EE514 Board:C_0603_1608Metric_Pad0.98x0.95mm_HandSolder
- L201, L202, L203: renamed from L?; footprint (none) -> EE514 Board:L_0603_1608Metric_Pad0.98x0.95mm_HandSolder
- Q201: renamed from Q?; footprint (none) -> EE514 Board:SOT-343_2.0x1.25mm_P1.3mm
- R201: renamed from R?; footprint (none) -> EE514 Board:R_0603_1608Metric_Pad0.98x0.95mm_HandSolder
Connections:
- net RF_IN: now reaches C201.2, L201.1
- net RF_OUT: now reaches C205.1
Changed lines of the file:
@@
 $Descr A4 11693 8268
 encoding utf-8
-Sheet 2 4
+Sheet 2 5
 Title ""
 Date ""
@@
 $EndDescr
 $Comp
-L Connector:Conn_Coaxial J?
-U 1 1 6196BC05
-P 850 3950
-F 0 "J?" H 778 4188 50  0000 C CNN
-F 1 "SMA" H 778 4097 50  0000 C CNN
-F 2 "" H 850 3950 50  0001 C CNN
-F 3 " ~" H 850 3950 50  0001 C CNN
-	1    850  3950
-	-1   0    0    -1
-$EndComp
-$Comp
-L Device:L L?
+L Device:L L201
 U 1 1 6196D3C1
 P 1700 4350
-F 0 "L?" H 1753 4396 50  0000 L CNN
+F 0 "L201" H 1753 4396 50  0000 L CNN
 F 1 "2.2nH" H 1753 4305 50  0000 L CNN
-F 2 "" H 1700 4350 50  0001 C CNN
+F 2 "EE514 Board:L_0603_1608Metric_Pad0.98x0.95mm_HandSolder" H 1700 4350 50  0001 C CNN
 F 3 "~" H 1700 4350 50  0001 C CNN
 	1    1700 4350
@@
 $EndComp
 $Comp
-L Device:C C?
+L Device:C C201
 U 1 1 6196E6E7
 P 2150 3950
-F 0 "C?" V 1898 3950 50  0000 C CNN
+F 0 "C201" V 1898 3950 50  0000 C CNN
 F 1 "2.2pF" V 1989 3950 50  0000 C CNN
-F 2 "" H 2188 3800 50  0001 C CNN
+F 2 "EE514 Board:C_0603_1608Metric_Pad0.98x0.95mm_HandSolder" H 2188 3800 50  0001 C CNN
 F 3 "~" H 2150 3950 50  0001 C CNN
 	1    2150 3950
@@
 $EndComp
 $Comp
-L Device:L L?
+L Device:L L202
 U 1 1 6196F279
 P 3600 4350
-F 0 "L?" H 3653 4396 50  0000 L CNN
+F 0 "L202" H 3653 4396 50  0000 L CNN
 F 1 "18nH" H 3653 4305 50  0000 L CNN
-F 2 "" H 3600 4350 50  0001 C CNN
+F 2 "EE514 Board:L_0603_1608Metric_Pad0.98x0.95mm_HandSolder" H 3600 4350 50  0001 C CNN
 F 3 "~" H 3600 4350 50  0001 C CNN
 	1    3600 4350
@@
 $EndComp
 $Comp
-L Device:C C?
+L Device:C C202
 U 1 1 6196F9F8
 P 3900 5050
-F 0 "C?" H 4015 5096 50  0000 L CNN
+F 0 "C202" H 4015 5096 50  0000 L CNN
 F 1 "7.5pF" H 4015 5005 50  0000 L CNN
-F 2 "" H 3938 4900 50  0001 C CNN
+F 2 "EE514 Board:C_0603_1608Metric_Pad0.98x0.95mm_HandSolder" H 3938 4900 50  0001 C CNN
 F 3 "~" H 3900 5050 50  0001 C CNN
 	1    3900 5050
@@
 $EndComp
 Wire Wire Line
-	1050 3950 1700 3950
-Wire Wire Line
 	2300 3950 3600 3950
 Wire Wire Line
@@
 Wire Wire Line
 	1700 4200 1700 3950
-Connection ~ 1700 3950
 Wire Wire Line
 	1700 3950 2000 3950
@@
 	3900 4800 3600 4800
 $Comp
-L power:GND #PWR?
+L power:GND #PWR0201
 U 1 1 61972909
 P 1700 4700
-F 0 "#PWR?" H 1700 4450 50  0001 C CNN
+F 0 "#PWR0201" H 1700 4450 50  0001 C CNN
 F 1 "GND" H 1705 4527 50  0000 C CNN
 F 2 "" H 1700 4700 50  0001 C CNN
@@
 $EndComp
 $Comp
-L power:GND #PWR?
+L power:GND #PWR0202
 U 1 1 61972BFE
 P 3900 5350
-F 0 "#PWR?" H 3900 5100 50  0001 C CNN
+F 0 "#PWR0202" H 3900 5100 50  0001 C CNN
 F 1 "GND" H 3905 5177 50  0000 C CNN
 F 2 "" H 3900 5350 50  0001 C CNN
@@
 V_BIAS_BASE
 $Comp
-L Device:R_US R?
+L Device:R_US R201
 U 1 1 61974774
 P 5100 3950
-F 0 "R?" V 4895 3950 50  0000 C CNN
+F 0 "R201" V 4895 3950 50  0000 C CNN
 F 1 "1.5" V 4986 3950 50  0000 C CNN
-F 2 "" V 5140 3940 50  0001 C CNN
+F 2 "EE514 Board:R_0603_1608Metric_Pad0.98x0.95mm_HandSolder" V 5140 3940 50  0001 C CNN
 F 3 "~" H 5100 3950 50  0001 C CNN
 	1    5100 3950
@@
 $EndComp
 $Comp
-L Device:C C?
+L Device:C C203
 U 1 1 619752CB
 P 5100 3350
-F 0 "C?" V 4848 3350 50  0000 C CNN
+F 0 "C203" V 4848 3350 50  0000 C CNN
 F 1 "7.5pF" V 4939 3350 50  0000 C CNN
-F 2 "" H 5138 3200 50  0001 C CNN
+F 2 "EE514 Board:C_0603_1608Metric_Pad0.98x0.95mm_HandSolder" H 5138 3200 50  0001 C CNN
 F 3 "~" H 5100 3350 50  0001 C CNN
 	1    5100 3350
@@
 Connection ~ 5600 3950
 $Comp
-L Device:L L?
+L Device:L L203
 U 1 1 619809E0
 P 8850 3850
-F 0 "L?" H 8903 3896 50  0000 L CNN
+F 0 "L203" H 8903 3896 50  0000 L CNN
 F 1 "3.9nH" H 8903 3805 50  0000 L CNN
-F 2 "" H 8850 3850 50  0001 C CNN
+F 2 "EE514 Board:L_0603_1608Metric_Pad0.98x0.95mm_HandSolder" H 8850 3850 50  0001 C CNN
 F 3 "~" H 8850 3850 50  0001 C CNN
 	1    8850 3850
@@
 	9150 4700 8850 4700
 $Comp
-L power:GND #PWR?
+L power:GND #PWR0204
 U 1 1 619823B5
 P 9150 5250
-F 0 "#PWR?" H 9150 5000 50  0001 C CNN
+F 0 "#PWR0204" H 9150 5000 50  0001 C CNN
 F 1 "GND" H 9155 5077 50  0000 C CNN
 F 2 "" H 9150 5250 50  0001 C CNN
@@
 	8850 3450 8850 3700
 $Comp
-L Device:C C?
+L Device:C C205
 U 1 1 6198398D
 P 9400 3450
-F 0 "C?" V 9148 3450 50  0000 C CNN
+F 0 "C205" V 9148 3450 50  0000 C CNN
 F 1 "3.9pF" V 9239 3450 50  0000 C CNN
-F 2 "" H 9438 3300 50  0001 C CNN
+F 2 "EE514 Board:C_0603_1608Metric_Pad0.98x0.95mm_HandSolder" H 9438 3300 50  0001 C CNN
 F 3 "~" H 9400 3450 50  0001 C CNN
 	1    9400 3450
@@
 	8850 3450 9250 3450
 Connection ~ 8850 3450
-$Comp
-L Connector:Conn_Coaxial J?
-U 1 1 61984484
-P 10600 3450
-F 0 "J?" H 10700 3425 50  0000 L CNN
-F 1 "SMA" H 10700 3334 50  0000 L CNN
-F 2 "" H 10600 3450 50  0001 C CNN
-F 3 " ~" H 10600 3450 50  0001 C CNN
-	1    10600 3450
-	1    0    0    -1
-$EndComp
 Wire Wire Line
 	9550 3450 10400 3450
-Wire Wire Line
-	10600 3650 10600 3900
-$Comp
-L power:GND #PWR?
-U 1 1 6198629A
-P 10600 3900
-F 0 "#PWR?" H 10600 3650 50  0001 C CNN
-F 1 "GND" H 10605 3727 50  0000 C CNN
-F 2 "" H 10600 3900 50  0001 C CNN
-F 3 "" H 10600 3900 50  0001 C CNN
-	1    10600 3900
-	1    0    0    -1
-$EndComp
-Wire Wire Line
-	850  4150 850  4400
-$Comp
-L power:GND #PWR?
-U 1 1 61986848
-P 850 4400
-F 0 "#PWR?" H 850 4150 50  0001 C CNN
-F 1 "GND" H 855 4227 50  0000 C CNN
-F 2 "" H 850 4400 50  0001 C CNN
-F 3 "" H 850 4400 50  0001 C CNN
-	1    850  4400
-	1    0    0    -1
-$EndComp
 Wire Notes Line
 	7750 2750 7750 4150
@@
 Input Matching \nNetwork\n
 $Comp
-L Device:C C?
+L Device:C C204
 U 1 1 619B560B
 P 9150 4950
-F 0 "C?" H 9265 4996 50  0000 L CNN
+F 0 "C204" H 9265 4996 50  0000 L CNN
 F 1 "7.5pF" H 9265 4905 50  0000 L CNN
-F 2 "" H 9188 4800 50  0001 C CNN
+F 2 "EE514 Board:C_0603_1608Metric_Pad0.98x0.95mm_HandSolder" H 9188 4800 50  0001 C CNN
 F 3 "~" H 9150 4950 50  0001 C CNN
 	1    9150 4950
@@
 $EndComp
 $Comp
-L EE514_Board:Q_NPN_BECE Q?
+L EE514_Board:Q_NPN_BECE Q201
 U 1 1 619B44AB
 P 6500 3950
-F 0 "Q?" H 6788 3996 50  0000 L CNN
+F 0 "Q201" H 6788 3996 50  0000 L CNN
 F 1 "BFP620" H 6788 3905 50  0000 L CNN
-F 2 "" H 6700 4050 50  0001 C CNN
+F 2 "EE514 Board:SOT-343_2.0x1.25mm_P1.3mm" H 6700 4050 50  0001 C CNN
 F 3 "~" H 6500 3950 50  0001 C CNN
 	1    6500 3950
@@
 	6600 4150 6600 4250
 $Comp
-L power:GND #PWR?
+L power:GND #PWR0203
 U 1 1 6197C06F
 P 6600 4400
-F 0 "#PWR?" H 6600 4150 50  0001 C CNN
+F 0 "#PWR0203" H 6600 4150 50  0001 C CNN
 F 1 "GND" H 6605 4227 50  0000 C CNN
 F 2 "" H 6600 4400 50  0001 C CNN
@@
 Text Notes 6850 4400 0    50   ~ 0
 Use two vias \nper pad
+Wire Wire Line
+	1700 3950 1150 3950
+Connection ~ 1700 3950
+Text HLabel 1150 3950 0    50   Input ~ 0
+RF_IN
+Text HLabel 10400 3450 2    50   Output ~ 0
+RF_OUT
 $EndSCHEMATC
