File: EE514 Board/EE514 Board.sch (KiCad schematic (older format))
At the start: 0 parts

Commit message: Layout finished, updating silkscreen...
Parts:
- added FL101: BPF-2, EE514 Board:Filter_2.0GHz_Bandpass_Edge-Coupled, symbol EE514_Board:BPF-2
- added J101: Screw_Terminal_01x02, TerminalBlock_TE-Connectivity:TerminalBlock_TE_282834-2_1x02_P2.54mm_Horizontal, symbol Connector:Screw_Terminal_01x02
- added J102, J103, J104, J105, J106: SMA, Connector_Coaxial:SMA_Molex_73251-1153_EdgeMount_Horizontal, symbol Connector:Conn_Coaxial
Connections:
- new net +5V: J101.2 (Pin_2)
- new net Amplifier/RF_IN: J103.1 (In)
- new net Amplifier/RF_OUT: J105.1 (In)
- new net FILT_IN: FL101.1 (IN), J102.1 (In)
- new net FILT_OUT: FL101.2 (OUT), J104.1 (In)
- new net GND: J101.1 (Pin_1), J102.2 (Ext), J103.2 (Ext), J104.2 (Ext), J105.2 (Ext), J106.2 (Ext)
- new net Oscillator/RF_OUT: J106.1 (In)
Other:
- note added: "Amplifier"
- note added: "Bandpass Filter"
- note added: "Oscillator"
- note added: "Power Input"
